File: current_sensor.kicad_pcb (KiCad board)
At the start: 2 copper layers, 14.7 x 12.2 mm, 5 parts, among them J3 Conn_01x03_Male, U1 ACS781xLRTR-100B

Commit message: hopefully this makes copper be copper
Parts:
- renumbered C2 to Cf, R1 to Rf
Routing:
- net +12V: track 0.00 -> 2.15 mm
- net -12V: track 0.00 -> 1.89 mm
Changed lines of the file:
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@@
     (pad_to_mask_clearance 0)
     (pcbplotparams
-      (layerselection 0x00010e8_ffffffff)
+      (layerselection 0x00010fc_ffffffff)
       (disableapertmacros false)
       (usegerberextensions true)
       (usegerberattributes true)
       (usegerberadvancedattributes true)
-      (creategerberjobfile true)
+      (creategerberjobfile false)
       (svguseinch false)
       (svgprecision 6)
@@
       (psa4output false)
       (plotreference true)
-      (plotvalue true)
+      (plotvalue false)
       (plotinvisibletext false)
       (sketchpadsonfab false)
-      (subtractmaskfromsilk false)
+      (subtractmaskfromsilk true)
       (outputformat 1)
       (mirror false)
@@
     (property "Sheetname" "")
     (attr smd)
-    (fp_text reference "R1" (at 0 1.524 270) (layer "F.SilkS")
+    (fp_text reference "Rf" (at -1.016 1.27 270) (layer "F.SilkS")
       (effects (font (size 1 1) (thickness 0.15)))
     )
@@
     (property "Sheetname" "")
     (attr smd)
-    (fp_text reference "U1" (at 0 0) (layer "F.SilkS")
+    (fp_text reference "U1" (at 1.778 -4.318) (layer "F.SilkS")
       (effects (font (size 1 1) (thickness 0.15)))
     )
@@
     (property "Sheetname" "")
     (attr smd)
-    (fp_text reference "C2" (at 2.54 0 180) (layer "F.SilkS")
+    (fp_text reference "Cf" (at 2.54 0 180) (layer "F.SilkS")
       (effects (font (size 1 1) (thickness 0.15)))
     )
@@
     (pad "3" smd roundrect (at 1.25 2.4 270) (size 0.8 1.6) (layers "B.Cu" "B.Paste" "B.Mask") (roundrect_rratio 0.25)
       (net 7 "GNDREF") (pinfunction "Pin_3") (pintype "passive"))
-    (pad "MP" smd roundrect (at -3.8 -0.5 270) (size 2.1 3) (layers "B.Cu" "B.Paste" "B.Mask") (roundrect_rratio 0.119048))
-    (pad "MP" smd roundrect (at 3.8 -0.5 270) (size 2.1 3) (layers "B.Cu" "B.Paste" "B.Mask") (roundrect_rratio 0.119048))
+    (pad "MP" smd roundrect (at -3.8 -0.5 270) (size 2.1 3) (layers "B.Cu" "B.Paste" "B.Mask") (roundrect_rratio 0.1190480952))
+    (pad "MP" smd roundrect (at 3.8 -0.5 270) (size 2.1 3) (layers "B.Cu" "B.Paste" "B.Mask") (roundrect_rratio 0.1190480952))
     (model "${KICAD6_3DMODEL_DIR}/Connector_Molex.3dshapes/Molex_PicoBlade_53261-0371_1x03-1MP_P1.25mm_Horizontal.wrl"
       (offset (xyz 0 0 0))
@@
     )
   )
-  (gr_line (start 202.438 90.424) (end 204.978 90.424) (layer "F.Cu") (width 1.75))
-  (gr_line (start 202.184 87.376) (end 204.724 87.376) (layer "F.Cu") (width 1.75))
   (gr_line (start 202.184 87.376) (end 204.724 87.376) (layer "F.Mask") (width 1.75))
   (gr_line (start 202.184 86.36) (end 202.184 81.28) (layer "F.Mask") (width 3))
@@
     (effects (font (size 0.75 0.75) (thickness 0.1875)) (justify mirror))
   )
-  (gr_text "ACS781" (at 208.28 92.456) (layer "F.SilkS")
+  (gr_text "ACS781" (at 208.28 92.71) (layer "F.SilkS")
     (effects (font (size 0.5 0.5) (thickness 0.12)))
   )
@@
   (segment (start 208.694 86.36) (end 210.312 86.36) (width 0.25) (layer "B.Cu") (net 1))
   (segment (start 212.852 90.7785) (end 212.5735 90.5) (width 0.25) (layer "F.Cu") (net 4))
-  (segment (start 206.756 87.542) (end 206.756 87.376) (width 0.25) (layer "F.Cu") (net 4))
-  (segment (start 209.714 90.5) (end 206.756 87.542) (width 0.25) (layer "F.Cu") (net 4))
+  (segment (start 208.014 88.9) (end 206.248 88.9) (width 0.25) (layer "F.Cu") (net 4))
+  (segment (start 209.614 90.5) (end 208.014 88.9) (width 0.25) (layer "F.Cu") (net 4))
   (segment (start 212.5735 90.5) (end 209.714 90.5) (width 0.25) (layer "F.Cu") (net 4))
-  (via (at 206.756 87.376) (size 0.8) (drill 0.4) (layers "F.Cu" "B.Cu") (net 4))
-  (segment (start 207.619538 88.392) (end 207.912 88.392) (width 0.25) (layer "B.Cu") (net 4))
-  (segment (start 206.756 87.376) (end 206.756 87.528462) (width 0.25) (layer "B.Cu") (net 4))
-  (segment (start 206.756 87.528462) (end 207.619538 88.392) (width 0.25) (layer "B.Cu") (net 4))
+  (segment (start 209.714 90.5) (end 209.614 90.5) (width 0.25) (layer "F.Cu") (net 4))
+  (via (at 206.248 88.9) (size 0.8) (drill 0.4) (layers "F.Cu" "B.Cu") (net 4))
+  (segment (start 206.756 88.392) (end 206.248 88.9) (width 0.25) (layer "B.Cu") (net 4))
+  (segment (start 207.912 88.392) (end 206.756 88.392) (width 0.25) (layer "B.Cu") (net 4))
+  (segment (start 204.864 87.4) (end 202.716 87.4) (width 1.5) (layer "F.Cu") (net 5))
   (via (at 202.692 85.852) (size 0.8) (drill 0.4) (layers "F.Cu" "B.Cu") (free) (net 5))
   (via (at 202.692 84.836) (size 0.8) (drill 0.4) (layers "F.Cu" "B.Cu") (free) (net 5))
@@
   (via (at 202.692 83.312) (size 0.8) (drill 0.4) (layers "F.Cu" "B.Cu") (free) (net 5))
   (via (at 201.168 83.312) (size 0.8) (drill 0.4) (layers "F.Cu" "B.Cu") (free) (net 5))
+  (segment (start 204.864 90.4) (end 202.97 90.4) (width 1.5) (layer "F.Cu") (net 6))
   (via (at 201.168 91.44) (size 0.8) (drill 0.4) (layers "F.Cu" "B.Cu") (free) (net 6))
   (via (at 202.692 91.948) (size 0.8) (drill 0.4) (layers "F.Cu" "B.Cu") (free) (net 6))

Commit message: symmetry
Other:
- board size 14.7 x 12.2 mm -> 14.7 x 13.1 mm
Changed lines of the file:
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@@
   )
   (gr_line (start 202.184 87.376) (end 204.724 87.376) (layer "F.Mask") (width 1.75))
-  (gr_line (start 202.184 86.36) (end 202.184 81.28) (layer "F.Mask") (width 3))
-  (gr_line (start 202.184 89.916) (end 202.184 95.504) (layer "F.Mask") (width 3))
+  (gr_line (start 202.184 86.614) (end 202.184 81.534) (layer "F.Mask") (width 3))
+  (gr_line (start 202.1332 91.186) (end 202.1332 96.774) (layer "F.Mask") (width 3))
   (gr_line (start 202.184 90.424) (end 204.724 90.424) (layer "F.Mask") (width 1.7))
-  (gr_rect (start 200.152 82.296) (end 214.884 94.488) (layer "Edge.Cuts") (width 0.1) (fill none))
-  (gr_text "Justin Bak" (at 206.248 93.472) (layer "B.SilkS")
+  (gr_rect (start 200.152 82.296) (end 214.884 95.4024) (layer "Edge.Cuts") (width 0.1) (fill none))
+  (gr_text "Justin Bak" (at 203.708 94.234) (layer "B.SilkS")
     (effects (font (size 0.75 0.75) (thickness 0.1875)) (justify mirror))
   )
@@
   (via (at 202.692 91.948) (size 0.8) (drill 0.4) (layers "F.Cu" "B.Cu") (free) (net 6))
   (via (at 201.676 92.456) (size 0.8) (drill 0.4) (layers "F.Cu" "B.Cu") (free) (net 6))
-  (via (at 202.184 89.916) (size 0.8) (drill 0.4) (layers "F.Cu" "B.Cu") (free) (net 6))
+  (via (at 201.676 93.3704) (size 0.8) (drill 0.4) (layers "F.Cu" "B.Cu") (free) (net 6))
   (via (at 202.692 92.964) (size 0.8) (drill 0.4) (layers "F.Cu" "B.Cu") (free) (net 6))
   (via (at 202.184 90.932) (size 0.8) (drill 0.4) (layers "F.Cu" "B.Cu") (free) (net 6))
@@
     (polygon
       (pts
-        (xy 215.392 87.884)
-        (xy 199.644 87.884)
+        (xy 215.392 88.138)
+        (xy 199.644 88.138)
         (xy 199.644 81.788)
         (xy 215.392 81.788)
@@
     (polygon
       (pts
-        (xy 215.392 94.996)
-        (xy 199.644 94.996)
-        (xy 199.644 88.392)
-        (xy 215.392 88.392)
+        (xy 215.392 95.504)
+        (xy 199.644 95.504)
+        (xy 199.644 89.662)
+        (xy 215.392 89.662)
       )
     )
@@
     (polygon
       (pts
-        (xy 215.392 94.996)
-        (xy 199.644 94.996)
+        (xy 215.392 95.504)
+        (xy 199.644 95.504)
         (xy 199.644 81.788)
         (xy 215.392 81.788)

Commit message: label the cap
Other:
- board text added: "0.1μF"
Changed lines of the file:
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@@
     (property "Sheetname" "")
     (attr smd)
-    (fp_text reference "C1" (at -2.54 0 180) (layer "F.SilkS")
+    (fp_text reference "C1" (at 0 1.27 270) (layer "F.SilkS")
       (effects (font (size 1 1) (thickness 0.15)))
     )
@@
     (effects (font (size 0.75 0.75) (thickness 0.1875)) (justify mirror))
   )
+  (gr_text "0.1μF" (at 212.598 92.202) (layer "F.SilkS")
+    (effects (font (size 1 1) (thickness 0.15)))
+  )
   (gr_text "ACS781" (at 208.28 92.71) (layer "F.SilkS")
